Commit message: add initial linear axis

File: assets/robot/openarm_v2.0/urdf/example/v2.urdf (robot description, URDF)
Before this commit: robot openarm_v20, 22 links, 21 joints
Links:
- added link openarm_chest_link0; collision mesh filename=package://openarm_description/assets/robot/openarm_v2.0/mes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 scale=0.001 0.001 0.001; visual mesh filename=package://openarm_description/assets/robot/openarm_v2.0/mes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 scale=1.0 1.0 1.0
- added link openarm_pedestal_link0; collision mesh filename=package://openarm_description/assets/robot/openarm_v2.0/mes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 scale=0.001 0.001 0.001; visual mesh filename=package://openarm_description/assets/robot/openarm_v2.0/mes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 scale=1.0 1.0 1.0
- link openarm_body_link0: geometry 
Joints:
- added joint openarm_body_pedestal_joint: type fixed, parent openarm_body_link0, child openarm_pedestal_link0, origin xyz=0.0 0.0 0.0 rpy=0.0 0.0 0.0
- added joint openarm_pedestal_chest_joint: type fixed, parent openarm_pedestal_link0, child openarm_chest_link0, origin xyz=0.0 0.0 0.0 rpy=0.0 0.0 0.0
- joint openarm_left_base_link_mount_joint: parent openarm_body_link0 -> openarm_chest_link0
- joint openarm_right_base_link_mount_joint: parent openarm_body_link0 -> openarm_chest_link0

File: assets/robot/openarm_v2.0/urdf/openarm_v20.urdf.xacro (robot description, xacro)
@@ -19,7 +19,9 @@
   <xacro:arg name="emit_grasp_frame" default="false" />
   <xacro:arg name="use_fake_hardware" default="true" />
+  <xacro:arg name="linear_axis_hardware_plugin" default="" />
   <xacro:property name="robot_root" value="$(find openarm_description)/assets/robot/openarm_v2.0" />
   <xacro:property name="config_root" value="${robot_root + '/config'}" />
   <xacro:property name="robot_preset_cfg" value="${xacro.load_yaml(config_root + '/robot_presets/' + '$(arg robot_preset)' + '.yaml')}" />
+  <xacro:property name="uses_linear_axis" value="${robot_preset_cfg['body']['config'] == 'body_linear_axis'}" />
   <xacro:openarm_v20_robot
     config_root="${config_root}"
@@ -41,3 +43,8 @@
     left_finger_mimic_multiplier="${pinch_finger_mimic_multiplier}"
     right_finger_mimic_multiplier="${pinch_finger_mimic_multiplier}" />
+  <xacro:if value="${uses_linear_axis}">
+    <xacro:openarm_linear_axis_ros2_control
+      use_fake_hardware="$(arg use_fake_hardware)"
+      linear_axis_hardware_plugin="$(arg linear_axis_hardware_plugin)" />
+  </xacro:if>
 </robot>

File: assets/robot/openarm_v2.0/urdf/ros2_control/openarm.bimanual.ros2_control.xacro (robot description, xacro)
@@ -13,4 +13,32 @@
 -->
 <robot xmlns:xacro="http://www.ros.org/wiki/xacro">
+<xacro:macro name="openarm_linear_axis_ros2_control"
+             params="use_fake_hardware linear_axis_hardware_plugin">
+  <ros2_control name="openarm_linear_axis_hardware_interface" type="system">
+    <hardware>
+      <xacro:if value="${use_fake_hardware}">
+        <plugin>mock_components/GenericSystem</plugin>
+        <param name="state_following_offset">0.0</param>
+      </xacro:if>
+      <xacro:unless value="${use_fake_hardware}">
+        <xacro:unless value="${linear_axis_hardware_plugin != ''}">
+          <xacro:property name="missing_linear_axis_plugin"
+                          value="${xacro.fatal('linear_axis_hardware_plugin must be set when use_fake_hardware is false')}"
+                          lazy_eval="false"/>
+        </xacro:unless>
+        <plugin>${linear_axis_hardware_plugin}</plugin>
+      </xacro:unless>
+    </hardware>
+    <joint name="openarm_linear_axis_joint">
+      <command_interface name="position"/>
+      <state_interface name="position">
+        <param name="initial_value">0.0</param>
+      </state_interface>
+      <state_interface name="velocity">
+        <param name="initial_value">0.0</param>
+      </state_interface>
+    </joint>
+  </ros2_control>
+</xacro:macro>
 <xacro:macro name="openarm_bimanual_ros2_control"
          params="arm_type

File: assets/robot/openarm_v2.0/urdf/utils/openarm_v20_robot.xacro (robot description, xacro)
@@ -23,7 +23,64 @@
     </xacro:unless>
   </xacro:macro>
+  <!-- Emit every non-root body link and its connection. -->
+  <xacro:macro name="openarm_v20_emit_body_links"
+    params="index topology link_name_map joint_prefix inertials visuals collisions reflect_x:=1 reflect_y:=1 reflect_z:=1 reflect_include_links:=^">
+    <xacro:if value="${index &lt; len(topology['links'])}">
+      <xacro:property name="source_link_name" value="${topology['links'][index]}" lazy_eval="false" />
+      <xacro:property
+        name="incoming_joint_names"
+        value="${[name for name in topology['joints'] if topology['joints'][name]['child'] == source_link_name]}"
+        lazy_eval="false" />
+      <xacro:openarm_v20_require
+        condition="${len(incoming_joint_names) == 1}"
+        message="${'Invalid body topology: link `%s` must have exactly one incoming joint.' % source_link_name}" />
+      <xacro:property name="source_joint_name" value="${incoming_joint_names[0]}" lazy_eval="false" />
+      <xacro:property name="joint_cfg" value="${topology['joints'][source_joint_name]}" lazy_eval="false" />
+      <xacro:property name="link_reflects" value="${source_link_name in reflect_include_links}" lazy_eval="false" />
+      <xacro:openarm_v20_require
+        condition="${joint_cfg['parent'] in link_name_map}"
+        message="${'Invalid body topology: joint `%s` references unknown parent `%s`.' % (source_joint_name, joint_cfg['parent'])}" />
+      <xacro:openarm_v20_emit_link
+        link_name="${link_name_map[source_link_name]}"
+        source_name="${source_link_name}"
+        inertials="${inertials}"
+        visuals="${visuals}"
+        collisions="${collisions}"
+        reflect_x="${reflect_x if link_reflects else 1}"
+        reflect_y="${reflect_y if link_reflects else 1}"
+        reflect_z="${reflect_z if link_reflects else 1}" />
+      <xacro:openarm_v20_emit_joint
+        joint_name="${joint_prefix}${source_joint_name}"
+        joint_type="${joint_cfg['type']}"
+        parent_link="${link_name_map[joint_cfg['parent']]}"
+        child_link="${link_name_map[source_link_name]}"
+        joint_origins="${dict()}"
+        joint_axes="${dict()}"
+        joint_limits="${dict()}"
+        source_name="${source_joint_name}"
+        origin_override="${joint_cfg['origin']}"
+        axis_override="${joint_cfg['axis'] if 'axis' in joint_cfg else 'none'}"
+        limit_override="${joint_cfg['limit'] if 'limit' in joint_cfg else 'none'}"
+        dynamics_override="${joint_cfg['dynamics'] if 'dynamics' in joint_cfg else 'none'}"
+        reflect_x="${reflect_x}"
+        reflect_y="${reflect_y}"
+        reflect_z="${reflect_z}" />
+      <xacro:openarm_v20_emit_body_links
+        index="${index + 1}"
+        topology="${topology}"
+        link_name_map="${link_name_map}"
+        joint_prefix="${joint_prefix}"
+        inertials="${inertials}"
+        visuals="${visuals}"
+        collisions="${collisions}"
+        reflect_x="${reflect_x}"
+        reflect_y="${reflect_y}"
+        reflect_z="${reflect_z}"
+        reflect_include_links="${reflect_include_links}" />
+    </xacro:if>
+  </xacro:macro>
   <!-- Emit the body component through the same mount contract used by other component types. -->
   <xacro:macro name="openarm_v20_body"
-    params="link_name connected_to mount_origin topology inertials visuals collisions reflect_x:=1 reflect_y:=1 reflect_z:=1 reflect_include_links:=^ skip_mount_joint:=false base_frame_shift:=none">
+    params="link_name connected_to mount_origin topology link_name_map link_prefix inertials visuals collisions reflect_x:=1 reflect_y:=1 reflect_z:=1 reflect_include_links:=^ skip_mount_joint:=false base_frame_shift:=none">
     <xacro:property name="base_link_name" value="${topology['links'][0]}" lazy_eval="false" />
     <xacro:property name="resolved_base_frame_shift" value="${base_frame_shift if base_frame_shift != 'none' else 'none'}" lazy_eval="false" />
@@ -46,4 +103,16 @@
       </joint>
     </xacro:unless>
+    <xacro:openarm_v20_emit_body_links
+      index="1"
+      topology="${topology}"
+      link_name_map="${link_name_map}"
+      joint_prefix="${link_prefix}"
+      inertials="${inertials}"
+      visuals="${visuals}"
+      collisions="${collisions}"
+      reflect_x="${reflect_x}"
+      reflect_y="${reflect_y}"
+      reflect_z="${reflect_z}"
+      reflect_include_links="${reflect_include_links}" />
   </xacro:macro>
   <!-- Load static resources and normalize product-specific preset data. -->
@@ -85,5 +154,5 @@
     <xacro:unless value="${source_type == 'sensor'}">
       <xacro:if value="${source_type == 'robot'}">
-        <xacro:property name="component_type" value="${component_config}" lazy_eval="false" />
+        <xacro:property name="component_type" value="${'body' if component_config == 'body_linear_axis' else component_config}" lazy_eval="false" />
         <xacro:property name="component_cfg_root" value="${config_root + '/' + component_config}" lazy_eval="false" />
       </xacro:if>
@@ -105,7 +174,10 @@
       <xacro:property name="component_visuals" value="${xacro.load_yaml(component_cfg_root + '/link/visuals.yaml')}" lazy_eval="false" />
       <xacro:property name="component_collisions" value="${xacro.load_yaml(component_cfg_root + '/link/collisions.yaml')}" lazy_eval="false" />
-      <xacro:property name="component_link_name_map" value="${dict(body_link0=component_cfg['link_name']) if component_type == 'body' else empty_dict}" lazy_eval="false" />
+      <xacro:property
+        name="component_link_name_map"
+        value="${dict([(source_link, component_cfg['link_name'] if source_link == component_topology['links'][0] else component_link_prefix + source_link) for source_link in component_topology['links']]) if component_type == 'body' else empty_dict}"
+        lazy_eval="false" />
       <xacro:property name="component_root_link_actual" value="${component_cfg['link_name'] if component_type == 'body' else (component_link_prefix + component_topology['links'][0])}" lazy_eval="false" />
-      <xacro:property name="component_default_mount_parent" value="${component_cfg['link_name'] if component_type == 'body' else (component_link_prefix + component_topology['links'][-1])}" lazy_eval="false" />
+      <xacro:property name="component_default_mount_parent" value="${component_link_name_map[component_topology['links'][-1]] if component_type == 'body' else (component_link_prefix + component_topology['links'][-1])}" lazy_eval="false" />
       <xacro:property name="component_supports_tip_collapse" value="${component_type == 'arm'}" lazy_eval="false" />
       <xacro:property
@@ -194,5 +266,5 @@
           message="${'Invalid robot preset: robot component `%s` uses unsupported product `%s`.' % (component_name, component_cfg['product'])}" />
         <xacro:openarm_v20_require
-          condition="${component_config in ['body', 'arm']}"
+          condition="${component_config in ['body', 'body_linear_axis', 'arm']}"
           message="${'Invalid robot preset: robot component `%s` has unsupported config `%s`.' % (component_name, component_config)}" />
       </xacro:if>
@@ -392,4 +464,6 @@
         mount_origin="${component_runtime['resolved_mount_origin']}"
         topology="${component_desc['topology']}"
+        link_name_map="${component_desc['link_name_map']}"
+        link_prefix="${component_desc['link_prefix']}"
         inertials="${component_desc['inertials']}"
         visuals="${component_desc['visuals']}"

File: assets/robot/openarm_v2.0/urdf/utils/openarm_v20_utils.xacro (robot description, xacro)
@@ -95,10 +95,15 @@
           </xacro:unless>
           <geometry>
-            <mesh
-              filename="${visual_cfg.geometry.mesh}"
-              scale="${reflect_x * visual_cfg.geometry.scale.x} ${reflect_y * visual_cfg.geometry.scale.y} ${reflect_z * visual_cfg.geometry.scale.z}" />
+            <xacro:if value="${'mesh' in visual_cfg.geometry}">
+              <mesh
+                filename="${visual_cfg.geometry.mesh}"
+                scale="${reflect_x * visual_cfg.geometry.scale.x} ${reflect_y * visual_cfg.geometry.scale.y} ${reflect_z * visual_cfg.geometry.scale.z}" />
+            </xacro:if>
+            <xacro:if value="${'box' in visual_cfg.geometry}">
+              <box size="${visual_cfg.geometry.box.x} ${visual_cfg.geometry.box.y} ${visual_cfg.geometry.box.z}" />
+            </xacro:if>
           </geometry>
           <material name="${link_name}_material">
-            <color rgba="0.752941176470588 0.752941176470588 0.752941176470588 1" />
+            <color rgba="${visual_cfg.material.rgba if 'material' in visual_cfg else '0.752941176470588 0.752941176470588 0.752941176470588 1'}" />
           </material>
         </visual>
@@ -114,7 +119,12 @@
           </xacro:unless>
           <geometry>
-            <mesh
-              filename="${collision_cfg.geometry.mesh}"
-              scale="${reflect_x * collision_cfg.geometry.scale.x} ${reflect_y * collision_cfg.geometry.scale.y} ${reflect_z * collision_cfg.geometry.scale.z}" />
+            <xacro:if value="${'mesh' in collision_cfg.geometry}">
+              <mesh
+                filename="${collision_cfg.geometry.mesh}"
+                scale="${reflect_x * collision_cfg.geometry.scale.x} ${reflect_y * collision_cfg.geometry.scale.y} ${reflect_z * collision_cfg.geometry.scale.z}" />
+            </xacro:if>
+            <xacro:if value="${'box' in collision_cfg.geometry}">
+              <box size="${collision_cfg.geometry.box.x} ${collision_cfg.geometry.box.y} ${collision_cfg.geometry.box.z}" />
+            </xacro:if>
           </geometry>
         </collision>
@@ -157,5 +167,5 @@
   </xacro:macro>
   <!-- Generic joint emitter with optional overrides for origin, axis, limits, and mimic. -->
-  <xacro:macro name="openarm_v20_emit_joint" params="joint_name joint_type parent_link child_link joint_origins joint_axes joint_limits reflect_x:=1 reflect_y:=1 reflect_z:=1 source_name:='' origin_override:=none axis_override:=none limit_override:=none mimic_override:=none mirror_limit_sign:=false frame_shift:=none">
+  <xacro:macro name="openarm_v20_emit_joint" params="joint_name joint_type parent_link child_link joint_origins joint_axes joint_limits reflect_x:=1 reflect_y:=1 reflect_z:=1 source_name:='' origin_override:=none axis_override:=none limit_override:=none mimic_override:=none dynamics_override:=none mirror_limit_sign:=false frame_shift:=none">
     <xacro:property name="source_joint_name" value="${source_name if source_name != '' else joint_name}" />
     <xacro:property name="joint_origin_cfg" value="${origin_override if origin_override != 'none' else joint_origins[source_joint_name].origin}" lazy_eval="false" />
@@ -200,4 +210,9 @@
           offset="${mimic_override['offset']}" />
       </xacro:if>
+      <xacro:if value="${joint_type != 'fixed' and dynamics_override != 'none'}">
+        <dynamics
+          damping="${dynamics_override['damping']}"
+          friction="${dynamics_override['friction']}" />
+      </xacro:if>
     </joint>
   </xacro:macro>
