Commit message: add 2d gripper camera frames

File: assets/robot/openarm_v2.0/urdf/openarm_v20.urdf.xacro (robot description, xacro)
@@ -15,4 +15,5 @@
   <xacro:include filename="$(find openarm_description)/assets/robot/openarm_v2.0/urdf/utils/openarm_v20_robot.xacro" />
   <xacro:include filename="$(find openarm_description)/assets/robot/openarm_v2.0/urdf/ros2_control/openarm.bimanual.ros2_control.xacro" />
+  <xacro:include filename="$(find openarm_description)/assets/robot/openarm_v2.0/urdf/sensors/openarm_b0495_wrist_cameras.xacro" />
   <xacro:arg name="robot_preset" default="default_bimanual" />
   <xacro:arg name="collapse_internal_empty_links" default="true" />
@@ -29,4 +30,18 @@
     collapse_internal_empty_links="$(arg collapse_internal_empty_links)"
     emit_grasp_frame="$(arg emit_grasp_frame)" />
+  <!-- A B0495 is part of each native pinch gripper. Emit it only for
+       enabled pinch-gripper components so single-arm presets remain valid. -->
+  <xacro:property name="primary_ee_cfg" value="${robot_preset_cfg['primary_arm_end_effector']}" />
+  <xacro:property name="secondary_ee_cfg" value="${robot_preset_cfg['secondary_arm_end_effector']}" />
+  <xacro:if value="${primary_ee_cfg['enabled'] and primary_ee_cfg['product'] == 'pinch_gripper'}">
+    <xacro:openarm_b0495_wrist_camera
+      side="${'left' if primary_ee_cfg['reflect']['y'] == -1 else 'right'}"
+      prefix="${primary_ee_cfg['prefix']}" />
+  </xacro:if>
+  <xacro:if value="${secondary_ee_cfg['enabled'] and secondary_ee_cfg['product'] == 'pinch_gripper'}">
+    <xacro:openarm_b0495_wrist_camera
+      side="${'left' if secondary_ee_cfg['reflect']['y'] == -1 else 'right'}"
+      prefix="${secondary_ee_cfg['prefix']}" />
+  </xacro:if>
   <xacro:property name="gains_file" value="${config_root}/arm/control/control_gains.yaml" />
   <xacro:property name="gains_dict" value="${xacro.load_yaml(gains_file)}" />

Commit message: move linear axis out

File: assets/robot/openarm_v2.0/urdf/openarm_v20.urdf.xacro (robot description, xacro)
@@ -23,9 +23,7 @@
   <xacro:arg name="right_can_interface" default="can0" />
   <xacro:arg name="can_fd" default="true" />
-  <xacro:arg name="linear_axis_hardware_plugin" default="" />
   <xacro:property name="robot_root" value="$(find openarm_description)/assets/robot/openarm_v2.0" />
   <xacro:property name="config_root" value="${robot_root + '/config'}" />
   <xacro:property name="robot_preset_cfg" value="${xacro.load_yaml(config_root + '/robot_presets/' + '$(arg robot_preset)' + '.yaml')}" />
-  <xacro:property name="uses_linear_axis" value="${robot_preset_cfg['body']['config'] == 'body_linear_axis'}" />
   <xacro:openarm_v20_robot
     config_root="${config_root}"
@@ -64,8 +62,3 @@
     left_finger_mimic_multiplier="${pinch_finger_mimic_multiplier}"
     right_finger_mimic_multiplier="${pinch_finger_mimic_multiplier}" />
-  <xacro:if value="${uses_linear_axis}">
-    <xacro:openarm_linear_axis_ros2_control
-      use_fake_hardware="$(arg use_fake_hardware)"
-      linear_axis_hardware_plugin="$(arg linear_axis_hardware_plugin)" />
-  </xacro:if>
 </robot>

File: assets/robot/openarm_v2.0/urdf/utils/openarm_v20_robot.xacro (robot description, xacro)
@@ -117,4 +117,63 @@
       reflect_include_links="${reflect_include_links}" />
   </xacro:macro>
+  <!-- OpenArm-owned chest mounted on a parameterized 60 x 60 mm aluminium profile. -->
+  <xacro:macro name="openarm_v20_body_aluminium_profile"
+    params="link_name connected_to mount_origin topology link_name_map inertials visuals collisions profile_height:=0.15 reflect_x:=1 reflect_y:=1 reflect_z:=1 reflect_include_links:=^ skip_mount_joint:=false base_frame_shift:=none">
+    <xacro:openarm_v20_require
+      condition="${profile_height > 0.0}"
+      message="Aluminium profile height must be positive." />
+    <xacro:property name="base_link_name" value="${topology['links'][0]}" lazy_eval="false" />
+    <xacro:property name="resolved_base_frame_shift" value="${base_frame_shift if base_frame_shift != 'none' else 'none'}" lazy_eval="false" />
+    <xacro:property name="base_link_reflects" value="${base_link_name in reflect_include_links}" lazy_eval="false" />
+    <xacro:openarm_v20_emit_link
+      link_name="${link_name}"
+      source_name="${base_link_name}"
+      inertials="${inertials}"
+      visuals="${visuals}"
+      collisions="${collisions}"
+      reflect_x="${reflect_x if base_link_reflects else 1}"
+      reflect_y="${reflect_y if base_link_reflects else 1}"
+      reflect_z="${reflect_z if base_link_reflects else 1}"
+      frame_shift="${resolved_base_frame_shift}" />
+    <xacro:unless value="${skip_mount_joint}">
+      <joint name="${link_name}_mount_joint" type="fixed">
+        <xacro:openarm_v20_emit_origin origin="${mount_origin}" reflect_x="1" reflect_y="1" reflect_z="1" reflect_position="false" />
+        <parent link="${connected_to}" />
+        <child link="${link_name}" />
+      </joint>
+    </xacro:unless>
+    <link name="${link_name_map['aluminium_profile_link']}">
+      <visual>
+        <geometry><box size="0.06 0.06 ${profile_height}" /></geometry>
+        <material name="aluminium_profile_material"><color rgba="0.22 0.22 0.22 1.0" /></material>
+      </visual>
+      <collision><geometry><box size="0.06 0.06 ${profile_height}" /></geometry></collision>
+      <inertial>
+        <mass value="${3.3333333333333335 * profile_height}" />
+        <inertia ixx="${(3.3333333333333335 * profile_height) * (0.06 * 0.06 + profile_height * profile_height) / 12.0}" ixy="0.0" ixz="0.0"
+                 iyy="${(3.3333333333333335 * profile_height) * (0.06 * 0.06 + profile_height * profile_height) / 12.0}" iyz="0.0" izz="${(3.3333333333333335 * profile_height) * (0.06 * 0.06 + 0.06 * 0.06) / 12.0}" />
+      </inertial>
+    </link>
+    <joint name="${link_name}_aluminium_profile_joint" type="fixed">
+      <parent link="${link_name}" />
+      <child link="${link_name_map['aluminium_profile_link']}" />
+      <origin xyz="0.0 0.0 ${profile_height / 2.0}" rpy="0.0 0.0 0.0" />
+    </joint>
+    <xacro:property name="chest_link_reflects" value="${'chest_link0' in reflect_include_links}" lazy_eval="false" />
+    <xacro:openarm_v20_emit_link
+      link_name="${link_name_map['chest_link0']}"
+      source_name="chest_link0"
+      inertials="${inertials}"
+      visuals="${visuals}"
+      collisions="${collisions}"
+      reflect_x="${reflect_x if chest_link_reflects else 1}"
+      reflect_y="${reflect_y if chest_link_reflects else 1}"
+      reflect_z="${reflect_z if chest_link_reflects else 1}" />
+    <joint name="${link_name}_aluminium_profile_chest_joint" type="fixed">
+      <parent link="${link_name_map['aluminium_profile_link']}" />
+      <child link="${link_name_map['chest_link0']}" />
+      <origin xyz="-0.01 0.0 0.009" rpy="0.0 0.0 0.0" />
+    </joint>
+  </xacro:macro>
   <!-- Load static resources and normalize product-specific preset data. -->
   <xacro:macro name="openarm_v20_load_component_descriptor"
@@ -155,5 +214,5 @@
     <xacro:unless value="${source_type == 'sensor'}">
       <xacro:if value="${source_type == 'robot'}">
-        <xacro:property name="component_type" value="${'body' if component_config == 'body_linear_axis' else component_config}" lazy_eval="false" />
+        <xacro:property name="component_type" value="${'body' if component_config == 'body_aluminium_profile' else component_config}" lazy_eval="false" />
         <xacro:property name="component_cfg_root" value="${config_root + '/' + component_config}" lazy_eval="false" />
       </xacro:if>
@@ -267,5 +326,5 @@
           message="${'Invalid robot preset: robot component `%s` uses unsupported product `%s`.' % (component_name, component_cfg['product'])}" />
         <xacro:openarm_v20_require
-          condition="${component_config in ['body', 'body_linear_axis', 'arm']}"
+          condition="${component_config in ['body', 'body_aluminium_profile', 'arm']}"
           message="${'Invalid robot preset: robot component `%s` has unsupported config `%s`.' % (component_name, component_config)}" />
       </xacro:if>
@@ -457,7 +516,25 @@
   <!-- Dispatch a resolved component to the concrete emitter for its type. -->
   <xacro:macro name="openarm_v20_emit_component_from_runtime"
-    params="component_desc component_runtime emit_grasp_frame:=false">
+    params="component_desc component_runtime emit_grasp_frame:=false aluminium_profile_height:=0.15">
     <xacro:property name="component_type" value="${component_runtime['component_type']}" lazy_eval="false" />
-    <xacro:if value="${component_type == 'body'}">
+    <xacro:if value="${component_type == 'body' and component_desc['config'] == 'body_aluminium_profile'}">
+      <xacro:openarm_v20_body_aluminium_profile
+        link_name="${component_desc['root_link_actual']}"
+        connected_to="${component_runtime['resolved_connected_to']}"
+        mount_origin="${component_runtime['resolved_mount_origin']}"
+        topology="${component_desc['topology']}"
+        link_name_map="${component_desc['link_name_map']}"
+        inertials="${component_desc['inertials']}"
+        visuals="${component_desc['visuals']}"
+        collisions="${component_desc['collisions']}"
+        profile_height="${aluminium_profile_height}"
+        reflect_x="${component_runtime['reflect_x']}"
+        reflect_y="${component_runtime['reflect_y']}"
+        reflect_z="${component_runtime['reflect_z']}"
+        reflect_include_links="${component_runtime['reflect_include_links']}"
+        skip_mount_joint="${component_runtime['skip_mount_joint']}"
+        base_frame_shift="${component_runtime['base_frame_shift']}" />
+    </xacro:if>
+    <xacro:if value="${component_type == 'body' and component_desc['config'] != 'body_aluminium_profile'}">
       <xacro:openarm_v20_body
         link_name="${component_desc['root_link_actual']}"
@@ -538,5 +615,5 @@
   <!-- Per-component orchestration: descriptor -> runtime resolution -> emission -> child recursion. -->
   <xacro:macro name="openarm_v20_emit_component_tree"
-    params="component_name components robot_preset config_root root_frame parent_desc:=none preloaded_desc:=none collapse_internal_empty_links:=false emit_grasp_frame:=false">
+    params="component_name components robot_preset config_root root_frame parent_desc:=none preloaded_desc:=none collapse_internal_empty_links:=false emit_grasp_frame:=false aluminium_profile_height:=0.15">
     <xacro:property name="none_value" value="${'none'}" lazy_eval="false" />
     <xacro:property name="component_cfg" value="${robot_preset[component_name]}" lazy_eval="false" />
@@ -563,5 +640,6 @@
       component_desc="${component_desc}"
       component_runtime="${component_runtime}"
-      emit_grasp_frame="${emit_grasp_frame}" />
+      emit_grasp_frame="${emit_grasp_frame}"
+      aluminium_profile_height="${aluminium_profile_height}" />
     <xacro:openarm_v20_emit_attached_components
       index="0"
@@ -575,9 +653,10 @@
       preloaded_component_desc="${component_runtime['collapse_child_desc']}"
       collapse_internal_empty_links="${collapse_internal_empty_links}"
-      emit_grasp_frame="${emit_grasp_frame}" />
+      emit_grasp_frame="${emit_grasp_frame}"
+      aluminium_profile_height="${aluminium_profile_height}" />
   </xacro:macro>
   <!-- Scan robot.components and emit every enabled child attached to the requested parent. -->
   <xacro:macro name="openarm_v20_emit_attached_components"
-    params="index components parent_component_name robot_preset config_root root_frame parent_desc:=none preloaded_component_name:=none preloaded_component_desc:=none collapse_internal_empty_links:=false emit_grasp_frame:=false">
+    params="index components parent_component_name robot_preset config_root root_frame parent_desc:=none preloaded_component_name:=none preloaded_component_desc:=none collapse_internal_empty_links:=false emit_grasp_frame:=false aluminium_profile_height:=0.15">
     <xacro:if value="${index &lt; len(components)}">
       <xacro:property name="none_value" value="${'none'}" lazy_eval="false" />
@@ -601,5 +680,6 @@
           preloaded_desc="${component_desc_override}"
           collapse_internal_empty_links="${collapse_internal_empty_links}"
-          emit_grasp_frame="${emit_grasp_frame}" />
+          emit_grasp_frame="${emit_grasp_frame}"
+          aluminium_profile_height="${aluminium_profile_height}" />
       </xacro:if>
       <xacro:openarm_v20_emit_attached_components
@@ -614,10 +694,11 @@
         preloaded_component_desc="${preloaded_component_desc}"
         collapse_internal_empty_links="${collapse_internal_empty_links}"
-        emit_grasp_frame="${emit_grasp_frame}" />
+        emit_grasp_frame="${emit_grasp_frame}"
+        aluminium_profile_height="${aluminium_profile_height}" />
     </xacro:if>
   </xacro:macro>
   <!-- Top-level robot emitter: validate the preset, emit the root frame, then expand the component tree. -->
   <xacro:macro name="openarm_v20_robot"
-    params="config_root robot_preset collapse_internal_empty_links:=false emit_grasp_frame:=false">
+    params="config_root robot_preset collapse_internal_empty_links:=false emit_grasp_frame:=false aluminium_profile_height:=0.15">
     <xacro:property name="robot_cfg" value="${robot_preset['robot']}" lazy_eval="false" />
     <xacro:property name="root_frame" value="${robot_cfg['root_frame']}" lazy_eval="false" />
@@ -635,5 +716,6 @@
       root_frame="${root_frame}"
       collapse_internal_empty_links="${collapse_internal_empty_links}"
-      emit_grasp_frame="${emit_grasp_frame}" />
+      emit_grasp_frame="${emit_grasp_frame}"
+      aluminium_profile_height="${aluminium_profile_height}" />
   </xacro:macro>
 </robot>
